Commit message: Replace RGB camera with depth camera and adjust position/tilt

File: install/arduinobot_description/share/arduinobot_description/urdf/arduinobot.urdf.xacro (robot description, xacro)
@@ -1,202 +1 @@
-<?xml version="1.0"?>
-<robot xmlns:xacro="http://www.ros.org/wiki/xacro" name="arduinobot">
-    <!-- Start GZ or Ignition depending on ROS 2 Version -->
-    <xacro:arg name="is_ignition" default="false"/>
-    <!-- Include Gazebo Parameters -->
-    <xacro:include filename="$(find arduinobot_description)/urdf/arduinobot_gazebo.xacro" />
-    <!-- Include ros2_control Plugins -->
-    <xacro:include filename="$(find arduinobot_description)/urdf/arduinobot_ros2_control.xacro" />
-    <!-- Useful XACRO Variables (Properties) -->
-    <xacro:property name="PI" value="3.14159265359" />
-    <xacro:property name="effort" value="30.0" />
-    <xacro:property name="velocity" value="10.0" />
-    <!-- Useful Macros -->
-    <xacro:macro name="default_inertial" params="mass">
-        <inertial>
-            <origin xyz="0 0 0" rpy="0 0 0"/>
-            <mass value="${mass}" />
-            <inertia ixx="1.0" ixy="0.0" ixz="0.0"
-                     iyy="1.0" iyz="0.0"
-                     izz="1.0" />
-        </inertial>
-    </xacro:macro>
-    <!-- Links -->
-    <link name="world"/>
-    <link name="base_link">
-        <xacro:default_inertial mass="1.0"/>
-        <visual>
-            <origin rpy="0 0 0" xyz="-0.5 -0.5 0"/>
-            <geometry>
-                <mesh filename="package://arduinobot_description/meshes/basement.STL" scale="0.01 0.01 0.01"/>
-            </geometry>
-        </visual>
-        <collision>
-            <origin rpy="0 0 0" xyz="-0.5 -0.5 0"/>
-            <geometry>
-                <mesh filename="package://arduinobot_description/meshes/basement.STL" scale="0.01 0.01 0.01"/>
-            </geometry>
-        </collision>
-    </link>
-    <link name="base_plate">
-        <xacro:default_inertial mass="0.1"/>
-        <visual>
-            <origin rpy="0 0 0" xyz="-0.39 -0.39 -0.56"/>
-            <geometry>
-                <mesh filename="package://arduinobot_description/meshes/base_plate.STL" scale="0.01 0.01 0.01"/>
-            </geometry>
-        </visual>
-        <collision>
-            <origin rpy="0 0 0" xyz="-0.39 -0.39 -0.56"/>
-            <geometry>
-                <mesh filename="package://arduinobot_description/meshes/base_plate.STL" scale="0.01 0.01 0.01"/>
-            </geometry>
-        </collision>
-    </link>
-    <link name="forward_drive_arm">
-        <xacro:default_inertial mass="0.1"/>
-        <visual>
-            <origin rpy=" 0 -${PI / 2} ${PI / 2}" xyz="0.19 0.06 -0.08"/>
-            <geometry>
-                <mesh filename="package://arduinobot_description/meshes/forward_drive_arm.STL" scale="0.01 0.01 0.01"/>
-            </geometry>
-        </visual>
-        <collision>
-            <origin rpy=" 0 -${PI / 2} ${PI / 2}" xyz="0.19 0.06 -0.08"/>
-            <geometry>
-                <mesh filename="package://arduinobot_description/meshes/forward_drive_arm.STL" scale="0.01 0.01 0.01"/>
-            </geometry>
-        </collision>
-    </link>
-    <link name="horizontal_arm">
-        <xacro:default_inertial mass="0.1"/>
-        <visual>
-            <origin rpy="${PI / 2} 0 ${PI / 2}" xyz="-0.03 -0.4 -0.06"/>
-            <geometry>
-                <mesh filename="package://arduinobot_description/meshes/horizontal_arm.STL" scale="0.01 0.01 0.01"/>
-            </geometry>
-        </visual>
-        <collision>
-            <origin rpy="${PI / 2} 0 ${PI / 2}" xyz="-0.03 -0.4 -0.06"/>
-            <geometry>
-                <mesh filename="package://arduinobot_description/meshes/horizontal_arm.STL" scale="0.01 0.01 0.01"/>
-            </geometry>
-        </collision>
-    </link>
-    <link name="claw_support">
-        <xacro:default_inertial mass="0.05"/>
-        <visual>
-            <origin rpy="0 0 ${PI / 2}" xyz="0 -0.05 -0.15"/>
-            <geometry>
-                <mesh filename="package://arduinobot_description/meshes/claw_support.STL" scale="0.01 0.01 0.01"/>
-            </geometry>
-        </visual>
-        <collision>
-            <origin rpy="0 0 ${PI / 2}" xyz="0 -0.05 -0.15"/>
-            <geometry>
-                <mesh filename="package://arduinobot_description/meshes/claw_support.STL" scale="0.01 0.01 0.01"/>
-            </geometry>
-        </collision>
-    </link>
-    <link name="gripper_right">
-        <xacro:default_inertial mass="0.01"/>
-        <visual>
-            <origin rpy="0 0 -${PI / 2}" xyz="-0.1 0.50 -0.1"/>
-            <geometry>
-                <mesh filename="package://arduinobot_description/meshes/right_finger.STL" scale="0.01 0.01 0.01"/>
-            </geometry>
-        </visual>
-        <collision>
-            <origin rpy="0 0 -${PI / 2}" xyz="-0.1 0.50 -0.1"/>
-            <geometry>
-                <mesh filename="package://arduinobot_description/meshes/right_finger.STL" scale="0.01 0.01 0.01"/>
-            </geometry>
-        </collision>
-    </link>
-    <link name="gripper_left">
-        <xacro:default_inertial mass="0.01"/>
-        <visual>
-            <origin rpy="0 0 -${PI / 2}" xyz="-0.04 0.50 -0.1"/>
-            <geometry>
-                <mesh filename="package://arduinobot_description/meshes/left_finger.STL" scale="0.01 0.01 0.01"/>
-            </geometry>
-        </visual>
-        <collision>
-            <origin rpy="0 0 -${PI / 2}" xyz="-0.04 0.50 -0.1"/>
-            <geometry>
-                <mesh filename="package://arduinobot_description/meshes/left_finger.STL" scale="0.01 0.01 0.01"/>
-            </geometry>
-        </collision>
-    </link>
-    <link name="rgb_camera">
-        <xacro:default_inertial mass="0.001"/>
-        <visual>
-            <origin rpy="-1.57 0 -1.57" xyz="-0.1 0.125 0.15"/>
-            <geometry>
-                <mesh filename="package://arduinobot_description/meshes/pi_camera.STL" scale="0.01 0.01 0.01"/>
-            </geometry>
-        </visual>
-        <collision>
-            <origin rpy="-1.57 0 -1.57" xyz="-0.1 0.125 0.15"/>
-            <geometry>
-                <mesh filename="package://arduinobot_description/meshes/pi_camera.STL" scale="0.01 0.01 0.01"/>
-            </geometry>
-        </collision>
-    </link>
-    <!-- Joints -->
-    <joint name="virtual_joint" type="fixed">
-        <parent link="world"/>
-        <child link="base_link"/>
-        <origin xyz="0 0 0" rpy="0 0 0"/>
-    </joint>
-    <joint name ="joint_1" type="revolute">
-        <parent link="base_link"/>
-        <child link = "base_plate"/>
-        <origin xyz="0 0 0.307"/>
-        <axis xyz="0 0 1"/>
-        <limit lower="-${PI / 2}" upper="${PI / 2}"
-               effort="${effort}" velocity="${velocity}"/>
-    </joint>
-    <joint name ="joint_2" type="revolute">
-        <parent link="base_plate"/>
-        <child link = "forward_drive_arm"/>
-        <origin xyz="-0.02 0 0.35"/>
-        <axis xyz="1 0 0"/>
-        <limit lower="-${PI / 2}" upper="${PI / 2}"
-                effort="${effort}" velocity="${velocity}"/>
-    </joint>
-    <joint name ="joint_3" type="revolute">
-        <parent link="forward_drive_arm"/>
-        <child link = "horizontal_arm"/>
-        <origin xyz="0 0 0.8"/>
-        <axis xyz="1 0 0"/>
-        <limit lower="-${PI / 2}" upper="${PI / 2}"
-               effort="${effort}" velocity="${velocity}"/>
-    </joint>
-    <joint name ="horizontal_arm_to_claw_support" type="fixed">
-        <parent link="horizontal_arm"/>
-        <child link = "claw_support"/>
-        <origin xyz="0 0.82 0"/>
-    </joint>
-    <joint name ="joint_4" type="revolute">
-        <parent link="claw_support"/>
-        <child link = "gripper_right"/>
-        <origin xyz="-0.04 0.13 -0.1"/>
-        <axis xyz="0 0 1"/>
-        <limit lower="-${PI / 2}" upper="0.0"
-               effort="${effort}" velocity="${velocity}"/>
-    </joint>
-    <joint name ="joint_5" type="revolute">
-        <parent link="claw_support"/>
-        <child link = "gripper_left"/>
-        <origin xyz="-0.22 0.13 -0.1"/>
-        <axis xyz="0 0 1"/>
-        <limit lower="0.0" upper="${PI / 2}"
-               effort="${effort}" velocity="${velocity}"/>
-        <mimic joint="joint_4" multiplier="-1"/>
-    </joint>
-    <joint name ="rgb_camera_joint" type="fixed">
-        <parent link="claw_support"/>
-        <child link = "rgb_camera"/>
-        <origin xyz="-0.1 0.325 0.3" rpy="0 0.4 1.57"/>
-    </joint>
-</robot>
+/home/jashwanth/arduinobot_ws/src/arduinobot_description/urdf/arduinobot.urdf.xacro

File: install/arduinobot_description/share/arduinobot_description/urdf/arduinobot_gazebo.xacro (robot description, xacro)
@@ -1,49 +1 @@
-<?xml version="1.0"?>
-<robot xmlns:xacro="http://www.ros.org/wiki/xacro" name="arduinobot">
-  <!-- ROS 2 Control -->
-  <gazebo>
-    <!-- ROS 2 Humble -->
-    <xacro:if value="$(arg is_ignition)">
-      <plugin filename="ign_ros2_control-system" name="ign_ros2_control::IgnitionROS2ControlPlugin">
-        <parameters>$(find arduinobot_controller)/config/arduinobot_controllers.yaml</parameters>
-      </plugin>
-      <plugin filename="ignition-gazebo-sensors-system" name="ignition::gazebo::systems::Sensors">
-        <render_engine>ogre2</render_engine>
-      </plugin>
-    </xacro:if>
-    <!-- ROS 2 Iron or above -->
-    <xacro:unless value="$(arg is_ignition)">
-      <plugin filename="gz_ros2_control-system" name="gz_ros2_control::GazeboSimROS2ControlPlugin">
-        <parameters>$(find arduinobot_controller)/config/arduinobot_controllers.yaml</parameters>
-      </plugin>
-      <plugin filename="gz-sim-sensors-system" name="gz::sim::systems::Sensors">
-        <render_engine>ogre2</render_engine>
-      </plugin>
-    </xacro:unless>
-  </gazebo>
-  <gazebo reference="rgb_camera">
-    <sensor name="camera" type="camera">
-        <always_on>true</always_on>
-        <update_rate>30.0</update_rate>
-        <visualize>true</visualize>
-        <topic>/image_raw</topic>
-        <gz_frame_id>/rgb_camera</gz_frame_id>
-        <camera name="camera">
-          <horizontal_fov>1.21126</horizontal_fov>
-          <image>
-            <width>2304</width>
-            <height>1296</height>
-            <format>R8G8B8</format>
-          </image>
-          <distortion>
-            <k1>0.0</k1>
-            <k2>0.0</k2>
-            <k3>0.0</k3>
-            <p1>0.0</p1>
-            <p2>0.0</p2>
-            <center>0.5 0.5</center>
-          </distortion>
-        </camera>
-    </sensor>
-  </gazebo>
-</robot>
+/home/jashwanth/arduinobot_ws/src/arduinobot_description/urdf/arduinobot_gazebo.xacro

File: install/arduinobot_description/share/arduinobot_description/urdf/arduinobot_ros2_control.xacro (robot description, xacro)
@@ -1,51 +1 @@
-<?xml version="1.0"?>
-<robot xmlns:xacro="http://www.ros.org/wiki/xacro" name="arduinobot">
-    <ros2_control name="RobotSystem" type="system">
-        <xacro:property name="PI" value="3.14159265359" />
-        <!-- ros2_control Gazebo -->
-        <!-- ROS 2 Humble -->
-        <xacro:if value="$(arg is_ignition)">
-            <hardware>
-                <plugin>ign_ros2_control/IgnitionSystem</plugin>
-            </hardware>
-        </xacro:if>
-        <!-- ROS 2 Iron or above -->
-        <xacro:unless value="$(arg is_ignition)">
-            <hardware>
-                <plugin>gz_ros2_control/GazeboSimSystem</plugin>
-            </hardware>
-        </xacro:unless>
-        <joint name="joint_1">
-            <command_interface name="position">
-            <param name="min">-${PI / 2}</param>
-            <param name="max">${PI / 2}</param>
-            </command_interface>
-            <state_interface name="position"/>
-        </joint>
-        <joint name="joint_2">
-            <command_interface name="position">
-            <param name="min">-${PI / 2}</param>
-            <param name="max">${PI / 2}</param>
-            </command_interface>
-            <state_interface name="position"/>
-        </joint>
-        <joint name="joint_3">
-            <command_interface name="position">
-            <param name="min">-${PI / 2}</param>
-            <param name="max">${PI / 2}</param>
-            </command_interface>
-            <state_interface name="position"/>
-        </joint>
-        <joint name="joint_4">
-            <command_interface name="position">
-            <param name="min">-${PI / 2}</param>
-            <param name="max">0.0</param>
-            </command_interface>
-            <state_interface name="position"/>
-        </joint>
-        <joint name="joint_5">
-            <param name="mimic">joint_4</param>
-            <param name="multiplier">-1</param>
-        </joint>
-    </ros2_control>
-</robot>
+/home/jashwanth/arduinobot_ws/src/arduinobot_description/urdf/arduinobot_ros2_control.xacro

File: src/arduinobot_description/urdf/arduinobot.urdf.xacro (robot description, xacro)
@@ -128,5 +128,5 @@
         </collision>
     </link>
-    <link name="rgb_camera">
+    <link name="depth_camera">
         <xacro:default_inertial mass="0.001"/>
         <visual>
@@ -195,8 +195,8 @@
         <mimic joint="joint_4" multiplier="-1"/>
     </joint>
-    <joint name ="rgb_camera_joint" type="fixed">
+    <joint name ="depth_camera_joint" type="fixed">
         <parent link="claw_support"/>
-        <child link = "rgb_camera"/>
-        <origin xyz="-0.1 0.325 0.3" rpy="0 0.4 1.57"/>
+        <child link = "depth_camera"/>
+        <origin xyz="-0.1 0.38 0.32" rpy="0 0.75 1.57"/>
     </joint>
 </robot>

File: src/arduinobot_description/urdf/arduinobot_gazebo.xacro (robot description, xacro)
@@ -22,26 +22,22 @@
     </xacro:unless>
   </gazebo>
-  <gazebo reference="rgb_camera">
-    <sensor name="camera" type="camera">
+  <gazebo reference="depth_camera">
+    <sensor name="depth_camera" type="depth_camera">
         <always_on>true</always_on>
         <update_rate>30.0</update_rate>
         <visualize>true</visualize>
-        <topic>/image_raw</topic>
-        <gz_frame_id>/rgb_camera</gz_frame_id>
-        <camera name="camera">
+        <topic>depth_camera</topic>
+        <gz_frame_id>depth_camera</gz_frame_id>
+        <camera name="depth_camera">
           <horizontal_fov>1.21126</horizontal_fov>
           <image>
-            <width>2304</width>
-            <height>1296</height>
-            <format>R8G8B8</format>
+            <width>640</width>
+            <height>480</height>
+            <format>R_FLOAT32</format>
           </image>
-          <distortion>
-            <k1>0.0</k1>
-            <k2>0.0</k2>
-            <k3>0.0</k3>
-            <p1>0.0</p1>
-            <p2>0.0</p2>
-            <center>0.5 0.5</center>
-          </distortion>
+          <clip>
+            <near>0.1</near>
+            <far>10.0</far>
+          </clip>
         </camera>
     </sensor>
