Commit message: Move gripper fingers forward to Y=0.35 for better reach

File: src/arduinobot_description/urdf/arduinobot.urdf.xacro (robot description, xacro)
@@ -181,5 +181,5 @@
         <parent link="claw_support"/>
         <child link = "gripper_right"/>
-        <origin xyz="-0.04 0.13 -0.1"/>
+        <origin xyz="-0.04 0.35 -0.1"/>
         <axis xyz="0 0 1"/>
         <limit lower="-${PI / 2}" upper="0.0"
@@ -189,5 +189,5 @@
         <parent link="claw_support"/>
         <child link = "gripper_left"/>
-        <origin xyz="-0.22 0.13 -0.1"/>
+        <origin xyz="-0.22 0.35 -0.1"/>
         <axis xyz="0 0 1"/>
         <limit lower="0.0" upper="${PI / 2}"

Commit message: Files cleanup: remove comments and unused code

File: src/arduinobot_description/urdf/arduinobot.urdf.xacro (robot description, xacro)
@@ -2,5 +2,5 @@
 <robot xmlns:xacro="http://www.ros.org/wiki/xacro" name="arduinobot">
     <!-- Start GZ or Ignition depending on ROS 2 Version -->
-    <xacro:arg name="is_ignition" default="false"/>
+    <xacro:arg name="is_ignition" default="false" />
     <!-- Include Gazebo Parameters -->
     <xacro:include filename="$(find arduinobot_description)/urdf/arduinobot_gazebo.xacro" />
@@ -14,189 +14,249 @@
     <xacro:macro name="default_inertial" params="mass">
         <inertial>
-            <origin xyz="0 0 0" rpy="0 0 0"/>
+            <origin xyz="0 0 0" rpy="0 0 0" />
             <mass value="${mass}" />
             <inertia ixx="1.0" ixy="0.0" ixz="0.0"
-                     iyy="1.0" iyz="0.0"
-                     izz="1.0" />
+                iyy="1.0" iyz="0.0"
+                izz="1.0" />
         </inertial>
     </xacro:macro>
     <!-- Links -->
-    <link name="world"/>
+    <link name="world" />
     <link name="base_link">
-        <xacro:default_inertial mass="1.0"/>
-        <visual>
-            <origin rpy="0 0 0" xyz="-0.5 -0.5 0"/>
-            <geometry>
-                <mesh filename="package://arduinobot_description/meshes/basement.STL" scale="0.01 0.01 0.01"/>
-            </geometry>
-        </visual>
-        <collision>
-            <origin rpy="0 0 0" xyz="-0.5 -0.5 0"/>
-            <geometry>
-                <mesh filename="package://arduinobot_description/meshes/basement.STL" scale="0.01 0.01 0.01"/>
+        <xacro:default_inertial mass="1.0" />
+        <visual>
+            <origin rpy="0 0 0" xyz="-0.5 -0.5 0" />
+            <geometry>
+                <mesh filename="package://arduinobot_description/meshes/basement.STL"
+                    scale="0.01 0.01 0.01" />
+            </geometry>
+        </visual>
+        <collision>
+            <origin rpy="0 0 0" xyz="-0.5 -0.5 0" />
+            <geometry>
+                <mesh filename="package://arduinobot_description/meshes/basement.STL"
+                    scale="0.01 0.01 0.01" />
             </geometry>
         </collision>
     </link>
     <link name="base_plate">
-        <xacro:default_inertial mass="0.1"/>
-        <visual>
-            <origin rpy="0 0 0" xyz="-0.39 -0.39 -0.56"/>
-            <geometry>
-                <mesh filename="package://arduinobot_description/meshes/base_plate.STL" scale="0.01 0.01 0.01"/>
-            </geometry>
-        </visual>
-        <collision>
-            <origin rpy="0 0 0" xyz="-0.39 -0.39 -0.56"/>
-            <geometry>
-                <mesh filename="package://arduinobot_description/meshes/base_plate.STL" scale="0.01 0.01 0.01"/>
+        <xacro:default_inertial mass="0.1" />
+        <visual>
+            <origin rpy="0 0 0" xyz="-0.39 -0.39 -0.56" />
+            <geometry>
+                <mesh filename="package://arduinobot_description/meshes/base_plate.STL"
+                    scale="0.01 0.01 0.01" />
+            </geometry>
+        </visual>
+        <collision>
+            <origin rpy="0 0 0" xyz="-0.39 -0.39 -0.56" />
+            <geometry>
+                <mesh filename="package://arduinobot_description/meshes/base_plate.STL"
+                    scale="0.01 0.01 0.01" />
             </geometry>
         </collision>
     </link>
     <link name="forward_drive_arm">
-        <xacro:default_inertial mass="0.1"/>
-        <visual>
-            <origin rpy=" 0 -${PI / 2} ${PI / 2}" xyz="0.19 0.06 -0.08"/>
-            <geometry>
-                <mesh filename="package://arduinobot_description/meshes/forward_drive_arm.STL" scale="0.01 0.01 0.01"/>
-            </geometry>
-        </visual>
-        <collision>
-            <origin rpy=" 0 -${PI / 2} ${PI / 2}" xyz="0.19 0.06 -0.08"/>
-            <geometry>
-                <mesh filename="package://arduinobot_description/meshes/forward_drive_arm.STL" scale="0.01 0.01 0.01"/>
+        <xacro:default_inertial mass="0.1" />
+        <visual>
+            <origin rpy=" 0 -${PI / 2} ${PI / 2}" xyz="0.19 0.06 -0.08" />
+            <geometry>
+                <mesh filename="package://arduinobot_description/meshes/forward_drive_arm.STL"
+                    scale="0.01 0.01 0.01" />
+            </geometry>
+        </visual>
+        <collision>
+            <origin rpy=" 0 -${PI / 2} ${PI / 2}" xyz="0.19 0.06 -0.08" />
+            <geometry>
+                <mesh filename="package://arduinobot_description/meshes/forward_drive_arm.STL"
+                    scale="0.01 0.01 0.01" />
             </geometry>
         </collision>
     </link>
     <link name="horizontal_arm">
-        <xacro:default_inertial mass="0.1"/>
-        <visual>
-            <origin rpy="${PI / 2} 0 ${PI / 2}" xyz="-0.03 -0.4 -0.06"/>
-            <geometry>
-                <mesh filename="package://arduinobot_description/meshes/horizontal_arm.STL" scale="0.01 0.01 0.01"/>
-            </geometry>
-        </visual>
-        <collision>
-            <origin rpy="${PI / 2} 0 ${PI / 2}" xyz="-0.03 -0.4 -0.06"/>
-            <geometry>
-                <mesh filename="package://arduinobot_description/meshes/horizontal_arm.STL" scale="0.01 0.01 0.01"/>
+        <xacro:default_inertial mass="0.1" />
+        <visual>
+            <origin rpy="${PI / 2} 0 ${PI / 2}" xyz="-0.03 -0.4 -0.06" />
+            <geometry>
+                <mesh filename="package://arduinobot_description/meshes/horizontal_arm.STL"
+                    scale="0.01 0.01 0.01" />
+            </geometry>
+        </visual>
+        <collision>
+            <origin rpy="${PI / 2} 0 ${PI / 2}" xyz="-0.03 -0.4 -0.06" />
+            <geometry>
+                <mesh filename="package://arduinobot_description/meshes/horizontal_arm.STL"
+                    scale="0.01 0.01 0.01" />
             </geometry>
         </collision>
     </link>
     <link name="claw_support">
-        <xacro:default_inertial mass="0.05"/>
-        <visual>
-            <origin rpy="0 0 ${PI / 2}" xyz="0 -0.05 -0.15"/>
-            <geometry>
-                <mesh filename="package://arduinobot_description/meshes/claw_support.STL" scale="0.01 0.01 0.01"/>
-            </geometry>
-        </visual>
-        <collision>
-            <origin rpy="0 0 ${PI / 2}" xyz="0 -0.05 -0.15"/>
-            <geometry>
-                <mesh filename="package://arduinobot_description/meshes/claw_support.STL" scale="0.01 0.01 0.01"/>
+        <xacro:default_inertial mass="0.05" />
+        <visual>
+            <origin rpy="0 0 ${PI / 2}" xyz="0 -0.05 -0.15" />
+            <geometry>
+                <mesh filename="package://arduinobot_description/meshes/claw_support.STL"
+                    scale="0.01 0.01 0.01" />
+            </geometry>
+        </visual>
+        <collision>
+            <origin rpy="0 0 ${PI / 2}" xyz="0 -0.05 -0.15" />
+            <geometry>
+                <mesh filename="package://arduinobot_description/meshes/claw_support.STL"
+                    scale="0.01 0.01 0.01" />
             </geometry>
         </collision>
     </link>
     <link name="gripper_right">
-        <xacro:default_inertial mass="0.01"/>
-        <visual>
-            <origin rpy="0 0 -${PI / 2}" xyz="-0.1 0.50 -0.1"/>
-            <geometry>
-                <mesh filename="package://arduinobot_description/meshes/right_finger.STL" scale="0.01 0.01 0.01"/>
-            </geometry>
-        </visual>
-        <collision>
-            <origin rpy="0 0 -${PI / 2}" xyz="-0.1 0.50 -0.1"/>
-            <geometry>
-                <mesh filename="package://arduinobot_description/meshes/right_finger.STL" scale="0.01 0.01 0.01"/>
-            </geometry>
+        <xacro:default_inertial mass="0.01" />
+        <visual>
+            <origin rpy="0 0 -${PI / 2}" xyz="-0.1 0.50 -0.1" />
+            <geometry>
+                <mesh filename="package://arduinobot_description/meshes/right_finger.STL"
+                    scale="0.01 0.01 0.01" />
+            </geometry>
+        </visual>
+        <collision>
+            <origin rpy="0 0 -${PI / 2}" xyz="-0.1 0.50 -0.1" />
+            <geometry>
+                <mesh filename="package://arduinobot_description/meshes/right_finger.STL"
+                    scale="0.01 0.01 0.01" />
+            </geometry>
+            <surface>
+                <friction>
+                    <ode>
+                        <mu>50.0</mu>
+                        <mu2>50.0</mu2>
+                    </ode>
+                </friction>
+                <contact>
+                    <ode>
+                        <kp>1e10</kp>
+                        <kd>100</kd>
+                    </ode>
+                </contact>
+            </surface>
         </collision>
     </link>
     <link name="gripper_left">
-        <xacro:default_inertial mass="0.01"/>
-        <visual>
-            <origin rpy="0 0 -${PI / 2}" xyz="-0.04 0.50 -0.1"/>
-            <geometry>
-                <mesh filename="package://arduinobot_description/meshes/left_finger.STL" scale="0.01 0.01 0.01"/>
-            </geometry>
-        </visual>
-        <collision>
-            <origin rpy="0 0 -${PI / 2}" xyz="-0.04 0.50 -0.1"/>
-            <geometry>
-                <mesh filename="package://arduinobot_description/meshes/left_finger.STL" scale="0.01 0.01 0.01"/>
-            </geometry>
-        </collision>
+        <xacro:default_inertial mass="0.01" />
+        <visual>
+            <origin rpy="0 0 -${PI / 2}" xyz="-0.04 0.50 -0.1" />
+            <geometry>
+                <mesh filename="package://arduinobot_description/meshes/left_finger.STL"
+                    scale="0.01 0.01 0.01" />
+            </geometry>
+        </visual>
+        <collision>
+            <origin rpy="0 0 -${PI / 2}" xyz="-0.04 0.50 -0.1" />
+            <geometry>
+                <mesh filename="package://arduinobot_description/meshes/left_finger.STL"
+                    scale="0.01 0.01 0.01" />
+            </geometry>
+            <surface>
+                <friction>
+                    <ode>
+                        <mu>50.0</mu>
+                        <mu2>50.0</mu2>
+                    </ode>
+                </friction>
+                <contact>
+                    <ode>
+                        <kp>1e10</kp>
+                        <kd>100</kd>
+                    </ode>
+                </contact>
+            </surface>
+        </collision>
+    </link>
+    <link name="tcp_link">
+        <xacro:default_inertial mass="0.0001" />
     </link>
     <link name="depth_camera">
-        <xacro:default_inertial mass="0.001"/>
-        <visual>
-            <origin rpy="-1.57 0 -1.57" xyz="-0.1 0.125 0.15"/>
-            <geometry>
-                <mesh filename="package://arduinobot_description/meshes/pi_camera.STL" scale="0.01 0.01 0.01"/>
-            </geometry>
-        </visual>
-        <collision>
-            <origin rpy="-1.57 0 -1.57" xyz="-0.1 0.125 0.15"/>
-            <geometry>
-                <mesh filename="package://arduinobot_description/meshes/pi_camera.STL" scale="0.01 0.01 0.01"/>
-            </geometry>
-        </collision>
+        <xacro:default_inertial mass="0.001" />
+        <visual>
+            <origin rpy="-1.57 0 -1.57" xyz="-0.1 0.125 0.15" />
+            <geometry>
+                <mesh filename="package://arduinobot_description/meshes/pi_camera.STL"
+                    scale="0.01 0.01 0.01" />
+            </geometry>
+        </visual>
+        <collision>
+            <origin rpy="-1.57 0 -1.57" xyz="-0.1 0.125 0.15" />
+            <geometry>
+                <mesh filename="package://arduinobot_description/meshes/pi_camera.STL"
+                    scale="0.01 0.01 0.01" />
+            </geometry>
+        </collision>
+    </link>
+    <link name="depth_camera_optical">
+        <xacro:default_inertial mass="0.0001" />
     </link>
     <!-- Joints -->
     <joint name="virtual_joint" type="fixed">
-        <parent link="world"/>
-        <child link="base_link"/>
-        <origin xyz="0 0 0" rpy="0 0 0"/>
-    </joint>
-    <joint name ="joint_1" type="revolute">
-        <parent link="base_link"/>
-        <child link = "base_plate"/>
-        <origin xyz="0 0 0.307"/>
-        <axis xyz="0 0 1"/>
+        <parent link="world" />
+        <child link="base_link" />
+        <origin xyz="0 0 0" rpy="0 0 0" />
+    </joint>
+    <joint name="joint_1" type="revolute">
+        <parent link="base_link" />
+        <child link="base_plate" />
+        <origin xyz="0 0 0.307" />
+        <axis xyz="0 0 1" />
         <limit lower="-${PI / 2}" upper="${PI / 2}"
-               effort="${effort}" velocity="${velocity}"/>
-    </joint>
-    <joint name ="joint_2" type="revolute">
-        <parent link="base_plate"/>
-        <child link = "forward_drive_arm"/>
-        <origin xyz="-0.02 0 0.35"/>
-        <axis xyz="1 0 0"/>
+            effort="${effort}" velocity="${velocity}" />
+    </joint>
+    <joint name="joint_2" type="revolute">
+        <parent link="base_plate" />
+        <child link="forward_drive_arm" />
+        <origin xyz="-0.02 0 0.35" />
+        <axis xyz="1 0 0" />
         <limit lower="-${PI / 2}" upper="${PI / 2}"
-                effort="${effort}" velocity="${velocity}"/>
-    </joint>
-    <joint name ="joint_3" type="revolute">
-        <parent link="forward_drive_arm"/>
-        <child link = "horizontal_arm"/>
-        <origin xyz="0 0 0.8"/>
-        <axis xyz="1 0 0"/>
+            effort="${effort}" velocity="${velocity}" />
+    </joint>
+    <joint name="joint_3" type="revolute">
+        <parent link="forward_drive_arm" />
+        <child link="horizontal_arm" />
+        <origin xyz="0 0 0.8" />
+        <axis xyz="1 0 0" />
         <limit lower="-${PI / 2}" upper="${PI / 2}"
-               effort="${effort}" velocity="${velocity}"/>
-    </joint>
-    <joint name ="horizontal_arm_to_claw_support" type="fixed">
-        <parent link="horizontal_arm"/>
-        <child link = "claw_support"/>
-        <origin xyz="0 0.82 0"/>
-    </joint>
-    <joint name ="joint_4" type="revolute">
-        <parent link="claw_support"/>
-        <child link = "gripper_right"/>
-        <origin xyz="-0.04 0.35 -0.1"/>
-        <axis xyz="0 0 1"/>
+            effort="${effort}" velocity="${velocity}" />
+    </joint>
+    <joint name="horizontal_arm_to_claw_support" type="fixed">
+        <parent link="horizontal_arm" />
+        <child link="claw_support" />
+        <origin xyz="0 0.82 0" />
+    </joint>
+    <joint name="joint_4" type="revolute">
+        <parent link="claw_support" />
+        <child link="gripper_right" />
+        <origin xyz="-0.04 0.35 -0.1" />
+        <axis xyz="0 0 1" />
         <limit lower="-${PI / 2}" upper="0.0"
-               effort="${effort}" velocity="${velocity}"/>
-    </joint>
-    <joint name ="joint_5" type="revolute">
-        <parent link="claw_support"/>
-        <child link = "gripper_left"/>
-        <origin xyz="-0.22 0.35 -0.1"/>
-        <axis xyz="0 0 1"/>
+            effort="${effort}" velocity="${velocity}" />
+    </joint>
+    <joint name="joint_5" type="revolute">
+        <parent link="claw_support" />
+        <child link="gripper_left" />
+        <origin xyz="-0.22 0.35 -0.1" />
+        <axis xyz="0 0 1" />
         <limit lower="0.0" upper="${PI / 2}"
-               effort="${effort}" velocity="${velocity}"/>
-        <mimic joint="joint_4" multiplier="-1"/>
-    </joint>
-    <joint name ="depth_camera_joint" type="fixed">
-        <parent link="claw_support"/>
-        <child link = "depth_camera"/>
-        <origin xyz="-0.1 0.38 0.32" rpy="0 0.75 1.57"/>
+            effort="${effort}" velocity="${velocity}" />
+        <mimic joint="joint_4" multiplier="-1" />
+    </joint>
+    <joint name="claw_support_to_tcp" type="fixed">
+        <parent link="claw_support" />
+        <child link="tcp_link" />
+        <origin xyz="-0.19 0.45 0.218" rpy="0 0 0" />
+    </joint>
+    <joint name="depth_camera_joint" type="fixed">
+        <parent link="claw_support" />
+        <child link="depth_camera" />
+        <origin xyz="-0.1 0.38 0.32" rpy="0 0.75 1.57079632679" />
+    </joint>
+    <joint name="depth_camera_optical_joint" type="fixed">
+        <parent link="depth_camera" />
+        <child link="depth_camera_optical" />
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
File: src/arduinobot_description/urdf/arduinobot_gazebo.xacro (robot description, xacro)
@@ -24,21 +24,21 @@
   <gazebo reference="depth_camera">
     <sensor name="rgbd_camera" type="rgbd_camera">
-        <always_on>true</always_on>
-        <update_rate>30.0</update_rate>
-        <visualize>true</visualize>
-        <topic>rgbd_camera</topic>
-        <gz_frame_id>/depth_camera</gz_frame_id>
-        <camera name="rgbd_camera">
-          <horizontal_fov>1.21126</horizontal_fov>
-          <image>
-            <width>640</width>
-            <height>480</height>
-            <format>R8G8B8</format>
-          </image>
-          <clip>
-            <near>0.1</near>
-            <far>10.0</far>
-          </clip>
-        </camera>
+      <always_on>true</always_on>
+      <update_rate>30.0</update_rate>
+      <visualize>true</visualize>
+      <topic>rgbd_camera</topic>
+      <gz_frame_id>depth_camera_optical</gz_frame_id>
+      <camera name="rgbd_camera">
+        <horizontal_fov>1.21126</horizontal_fov>
+        <image>
+          <width>640</width>
+          <height>480</height>
+          <format>R8G8B8</format>
+        </image>
+        <clip>
+          <near>0.1</near>
+          <far>10.0</far>
+        </clip>
+      </camera>
     </sensor>
   </gazebo>

File: src/arduinobot_description/urdf/arduinobot_ros2_control.xacro (robot description, xacro)
@@ -18,29 +18,29 @@
         <joint name="joint_1">
             <command_interface name="position">
-            <param name="min">-${PI / 2}</param>
-            <param name="max">${PI / 2}</param>
+                <param name="min">-${PI / 2}</param>
+                <param name="max">${PI / 2}</param>
             </command_interface>
-            <state_interface name="position"/>
+            <state_interface name="position" />
         </joint>
         <joint name="joint_2">
             <command_interface name="position">
-            <param name="min">-${PI / 2}</param>
-            <param name="max">${PI / 2}</param>
+                <param name="min">-${PI / 2}</param>
+                <param name="max">${PI / 2}</param>
             </command_interface>
-            <state_interface name="position"/>
+            <state_interface name="position" />
         </joint>
         <joint name="joint_3">
             <command_interface name="position">
-            <param name="min">-${PI / 2}</param>
-            <param name="max">${PI / 2}</param>
+                <param name="min">-${PI / 2}</param>
+                <param name="max">${PI / 2}</param>
             </command_interface>
-            <state_interface name="position"/>
+            <state_interface name="position" />
         </joint>
         <joint name="joint_4">
             <command_interface name="position">
-            <param name="min">-${PI / 2}</param>
-            <param name="max">0.0</param>
+                <param name="min">-${PI / 2}</param>
+                <param name="max">0.0</param>
             </command_interface>
-            <state_interface name="position"/>
+            <state_interface name="position" />
         </joint>
         <joint name="joint_5">
